Commit message: create initial URDF model of a car, rzviz and gazebo sim launchers, update readme

File: src/jetson_car_description/urdf/jetson_car.urdf.xacro (robot description, xacro)
@@ -164,3 +164,19 @@
     <origin xyz="0 0 0.04" rpy="0 0 0"/>
   </joint>
+  <!-- ===== Gazebo ===== -->
+  <gazebo reference="base_link">
+    <material>Gazebo/Blue</material>
+    <mu1>0.8</mu1>
+    <mu2>0.8</mu2>
+  </gazebo>
+  <xacro:macro name="wheel_gazebo_friction" params="link_name">
+    <gazebo reference="${link_name}">
+      <mu1>1.0</mu1>
+      <mu2>1.0</mu2>
+    </gazebo>
+  </xacro:macro>
+  <xacro:wheel_gazebo_friction link_name="front_left_wheel"/>
+  <xacro:wheel_gazebo_friction link_name="front_right_wheel"/>
+  <xacro:wheel_gazebo_friction link_name="rear_left_wheel"/>
+  <xacro:wheel_gazebo_friction link_name="rear_right_wheel"/>
 </robot>

Commit message: add a simple sim control

File: src/jetson_car_description/urdf/jetson_car.urdf.xacro (robot description, xacro)
@@ -180,3 +180,34 @@
   <xacro:wheel_gazebo_friction link_name="rear_left_wheel"/>
   <xacro:wheel_gazebo_friction link_name="rear_right_wheel"/>
+  <ros2_control name="GazeboSimSystem" type="system">
+    <hardware>
+      <plugin>gz_ros2_control/GazeboSimSystem</plugin>
+    </hardware>
+    <joint name="rear_left_drive_joint">
+      <command_interface name="velocity"/>    <!-- drive: speed command -->
+      <state_interface name="position"/>
+      <state_interface name="velocity"/>
+    </joint>
+    <joint name="rear_right_drive_joint">
+      <command_interface name="velocity"/>
+      <state_interface name="position"/>
+      <state_interface name="velocity"/>
+    </joint>
+    <joint name="front_left_steer_joint">
+      <command_interface name="position"/>    <!-- steer: angle command -->
+      <state_interface name="position"/>
+      <state_interface name="velocity"/>
+    </joint>
+    <joint name="front_right_steer_joint">
+      <command_interface name="position"/>
+      <state_interface name="position"/>
+      <state_interface name="velocity"/>
+    </joint>
+  </ros2_control>
+  <gazebo>
+    <plugin filename="gz_ros2_control-system"
+            name="gz_ros2_control::GazeboSimROS2ControlPlugin">
+      <parameters>$(find jetson_car_description)/config/controllers.yaml</parameters>
+    </plugin>
+  </gazebo>
 </robot>
